File: pcb/Doorbell2Thread.kicad_pcb (KiCad board)
At the start: 2 copper layers, 29 x 39 mm, 19 parts, among them J1 Klingel, Q1 2N7002, Q2 2N7002, SW1 TS-1088, SW2 TS-1088, U1 ESP32-H2-Zero, U2 LMS78_03-0.5R

Commit message: fix: add protection circuitry
The doorbell was killing the mosfets on the board so some protection was needed

feat: replaced the expensive LME78
This caused a major redesign of the whole board

fix: update to KiCad 10
Parts:
- added C1: 10u, Capacitor_SMD:C_0603_1608Metric, F.Cu at (120.8, 77.5)
- added C2: 10u, Capacitor_SMD:C_0603_1608Metric, F.Cu at (117.8, 77.5)
- added D1: MM3Z5V1, Diode_SMD:D_SOD-323, F.Cu at (121.0, 79.2)
- added D2: MM3Z5V1, Diode_SMD:D_SOD-323, F.Cu at (117.5, 79.2)
- added R1: 10k, Resistor_SMD:R_0402_1005Metric, F.Cu at (120.0, 81.2)
- added R2: 10k, Resistor_SMD:R_0402_1005Metric, F.Cu at (118.5, 81.2)
- added R5: 100k, Resistor_SMD:R_0402_1005Metric, F.Cu at (120.5, 71.2)
- added R6: 100k, Resistor_SMD:R_0402_1005Metric, F.Cu at (118.0, 71.2)
- R3: renamed from R1; footprint Resistor_SMD:R_0603_1608Metric -> Resistor_SMD:R_0402_1005Metric
- R4: renamed from R2; footprint Resistor_SMD:R_0603_1608Metric -> Resistor_SMD:R_0402_1005Metric
- U2: value LMS78_03-0.5R -> Mini DC-DC Module; footprint My_Footprints:LME78_1.0-Series -> My_Footprints:Mini DC-DC Module
- moved REF** 12.5 mm to (126.8, 76.8)
- moved G*** 12.4 mm to (133.2, 76.2)
- moved Q2 10.9 mm to (117.5, 73.8), turned to 90 degrees
- moved SW1 8.14 mm to (134.8, 89.0), turned to 90 degrees
- moved R3 6.75 mm to (120.5, 76.2), turned to 0 degrees
- moved C3 6.66 mm to (112.5, 72.2), turned to -90 degrees
- moved C4 6.66 mm to (112.5, 75.8), turned to 90 degrees
- moved SW2 6.52 mm to (134.8, 83.0), turned to 90 degrees
- moved Q1 6.17 mm to (121.0, 73.8), turned to 90 degrees
- moved U2 4.39 mm to (109.5, 72.8)
- moved R4 4.10 mm to (118.0, 76.2), turned to 180 degrees
- renumbered C1 to C3, C2 to C4, Q2 to Q1, Q1 to Q2
Connections:
- C3 pad 1: +9V -> /+9V
- C4 pad 1: +3V3 -> +5V
- J1 pad 3: +9V -> /+9V
- Q1 pad 1: /G3 -> /G1_{p}
- Q1 pad 3: /IO11 -> /IO13
- Q2 pad 1: /G1 -> /G3_{p}
- Q2 pad 3: /IO10 -> /IO14
- R3 pad 1: /G1 -> /G1_{p}
- R4 pad 1: /G3 -> /G3_{p}
- SW1 pad 2: /IO10 -> /IO13
- SW2 pad 2: /IO11 -> /IO14
- U1 pad 1: unconnected-(U1-5V-Pad1) -> +5V
- U1 pad 10: /IO10 -> unconnected-(U1-GPIO10-Pad10)
- U1 pad 11: /IO11 -> unconnected-(U1-GPIO11-Pad11)
- U1 pad 13: unconnected-(U1-GPIO13-Pad13) -> /IO13
- U1 pad 14: unconnected-(U1-GPIO14-Pad14) -> /IO14
- U2 pad 1: +9V -> unconnected-(U2-EN-Pad1)
- U2 pad 2: GND -> /+9V
- U2 pad 3: +3V3 -> GND
Routing:
- net /IO13: track 0.00 -> 40.1 mm, vias 0 -> 2
- net /IO14: track 0.00 -> 29.7 mm, vias 0 -> 2
- net +5V: track 0.00 -> 27.5 mm, vias 0 -> 2
- net /+9V: track 0.00 -> 22.8 mm, vias 0 -> 1
- net /IO11: track 19.1 -> 0.00 mm, vias 1 -> 0
- net /IO10: track 17.1 -> 0.00 mm, vias 1 -> 0
- net +9V: track 16.8 -> 0.00 mm
- net /G3_{p}: track 0.00 -> 7.38 mm
- net /G1_{p}: track 0.00 -> 6.14 mm
- net /G3: track 10.7 -> 5.01 mm
- net +3V3: track 21.7 -> 17.2 mm, vias 1 -> 2
- net GND: track 3.73 -> 0.00 mm, vias 25 -> 42
- net /G1: track 9.08 -> 7.33 mm
- added copper zone on In1.Cu, net GND
- added copper zone on In2.Cu, net GND
Other:
- copper layers 2 -> 4
- board text added: "Doorbell 2Thread"
- board text added: "G1 IO13"
- board text added: "G3 IO14"
- board text removed: "Doorbell 2 Thread"
- board text removed: "G1/ IO10"
- board text removed: "G3/ IO11"
- board text removed: "OUT GND IN"
